Commit message: 模拟参数调节

File: src/unitree_ros2_sim/go1_sim/go1_description/xacro/const.xacro (robot description, xacro)
@@ -48,6 +48,6 @@
     <xacro:property name="calf_rotor_offset_z" value="0.0"/>
     <!-- joint limits -->
-    <xacro:property name="damping" value="0.01"/>
-    <xacro:property name="friction" value="0.2"/>
+    <xacro:property name="damping" value="0.5"/>
+    <xacro:property name="friction" value="1.0"/>
     <xacro:property name="hip_position_max" value="0.863"/>
     <xacro:property name="hip_position_min" value="-0.863"/>
