Commit message: sync

File: src/unitree_ros2_sim/go1_sim/go1_description/xacro/robot.xacro (robot description, xacro)
@@ -137,5 +137,5 @@
     <link name="laser_link">
         <collision>
-            <origin xyz="0.05 0 0.5" rpy="0 0 0"/>
+            <origin xyz="0.0 0 0.0" rpy="0 0 0"/>
             <geometry>
                 <cylinder radius="0.05" length="0.05"/>
