Commit message: add mid360

File: src/unitree_go2w_ros2/go2w_description/urdf/go2w_description.urdf.xacro (robot description, xacro)
@@ -384,5 +384,5 @@
         <scan>
           <horizontal>
-            <samples>180</samples>
+            <samples>18</samples>
             <resolution>1</resolution>
             <min_angle>-3.14159</min_angle>
@@ -390,5 +390,5 @@
           </horizontal>
           <vertical>
-            <samples>30</samples>
+            <samples>1</samples>
             <resolution>1</resolution>
             <min_angle>${-PI/2.0 + 1.0}</min_angle>
@@ -416,4 +416,9 @@
     </sensor>
   </gazebo>
+  <!-- =============== mid360 ============ -->
+  <xacro:include filename="$(find go2w_description)/urdf/sensor/mid360_gpu.xacro"/>
+  <xacro:mid360  name="livox_frame" parent="base" topic="/livox/lidar" imu_topic="/livox/imu" >
+    <origin xyz="0.07 0.0 0.10" rpy="0 0.5235987756 0"/>
+  </xacro:mid360>
   <!-- Camera -->
   <link name="camera">

Commit message: gpu lidar

File: src/unitree_go2w_ros2/go2w_description/urdf/go2w_description.urdf.xacro (robot description, xacro)
@@ -418,6 +418,6 @@
   <!-- =============== mid360 ============ -->
   <xacro:include filename="$(find go2w_description)/urdf/sensor/mid360_gpu.xacro"/>
-  <xacro:mid360  name="livox_frame" parent="base" topic="/livox/lidar" imu_topic="/livox/imu" >
-    <origin xyz="0.07 0.0 0.10" rpy="0 0.5235987756 0"/>
+  <xacro:mid360  name="livox_frame" parent="body" topic="/livox/lidar" imu_topic="/livox/imu" >
+    <origin xyz="0.3 0.0 0.10" rpy="0 0.5235987756 0"/>
   </xacro:mid360>
   <!-- Camera -->

File: src/unitree_go2w_ros2/go2w_description/urdf/sensor/mid360_cpu.xacro (robot description, xacro)
@@ -21,8 +21,8 @@
     </inertial>
   </xacro:macro>
-  <xacro:macro name="mid360" params="name:='' parent:= 'base_link' topic:='mid360' imu_topic:='/livox/imu' *origin ">
+  <xacro:macro name="mid360" params="name:='' parent:= 'body' topic:='mid360' imu_topic:='/livox/imu' *origin ">
     <link name="${name}">
       <visual>
-        <origin xyz="0.025 -0.0265 -0.025" rpy="${pi/2} 0 ${pi}"/>
+        <origin xyz="0.025 -0.0265 -0.025" rpy="${pi/2} 0 ${pi/2}"/>
         <geometry>
           <mesh filename="package://go2w_description/meshes/mid-360-scaled.dae"/>
@@ -30,5 +30,5 @@
       </visual>
   <collision>
-    <origin xyz="0.025 -0.0265 -0.025" rpy="${pi/2} 0 ${pi}"/>
+    <origin xyz="0.025 -0.0265 -0.025" rpy="${pi/2} 0 ${pi/2}"/>
     <geometry>
       <mesh filename="package://go2w_description/meshes/mid-360-scaled.dae"/>

File: src/unitree_go2w_ros2/go2w_description/urdf/sensor/mid360_gpu.xacro (robot description, xacro)
@@ -21,5 +21,5 @@
     </inertial>
   </xacro:macro>
-  <xacro:macro name="mid360" params="name:='' parent:= 'base' topic:='/livox/lidar' imu_topic:='/livox/imu' *origin ">
+  <xacro:macro name="mid360" params="name:='' parent:= 'body' topic:='/livox/lidar' imu_topic:='/livox/imu' *origin ">
     <link name="${name}">
       <visual>
@@ -60,5 +60,5 @@
           <scan>
             <horizontal>
-              <samples>360</samples>
+              <samples>720</samples>
               <resolution>1</resolution>
               <min_angle>${0}</min_angle>
@@ -66,5 +66,5 @@
             </horizontal>
             <vertical>
-              <samples>60</samples>
+              <samples>120</samples>
               <resolution>1</resolution>
               <min_angle>${-7.22/180*M_PI}</min_angle>
@@ -87,5 +87,5 @@
         <pose>0 0 0 0 0 0</pose>
         <always_on>true</always_on>
-        <update_rate>40</update_rate>
+        <update_rate>200</update_rate>
         <use_strict_rate>true</use_strict_rate>
         <visualize>false</visualize>

Commit message: ego planner可以输出栅格地图

File: src/unitree_go2w_ros2/go2w_description/urdf/go2w_description.urdf.xacro (robot description, xacro)
@@ -419,5 +419,6 @@
   <xacro:include filename="$(find go2w_description)/urdf/sensor/mid360_gpu.xacro"/>
   <xacro:mid360  name="livox_frame" parent="body" topic="/livox/lidar" imu_topic="/livox/imu" >
-    <origin xyz="0.3 0.0 0.10" rpy="0 0.5235987756 0"/>
+    <!-- <origin xyz="0.3 0.0 0.10" rpy="0 0.5235987756 0"/> -->
+    <origin xyz="0.3 0.0 0.10" rpy="0 0.0 0"/>
   </xacro:mid360>
   <!-- Camera -->
@@ -520,3 +521,25 @@
     </plugin>
   </gazebo>
+  <!-- Gazebo Odometry Publisher Plugin - 发布机器狗真实位姿 -->
+  <gazebo>
+    <plugin filename="libgazebo_odometry_publisher.so" name="odometry_publisher">
+      <!-- 发布频率 (Hz) -->
+      <update_rate>30</update_rate>
+      <!-- 参考坐标系 -->
+      <frame_name>odom</frame_name>
+      <!-- 机器狗本体坐标系 -->
+      <body_name>base_footprint</body_name>
+      <!-- 发布的话题名称 -->
+      <topic_name>/gazebo/tower/go2w/odometry</topic_name>
+      <!-- 坐标系设置 -->
+      <xyz_offset>0 0 0</xyz_offset>
+      <rpy_offset>0 0 0</rpy_offset>
+      <!-- 高斯噪声设置 (可选) -->
+      <gaussian_noise>0.001</gaussian_noise>
+      <!-- 是否发布tf变换 -->
+      <publish_tf>true</publish_tf>
+      <!-- 坐标系前缀 -->
+      <frame_prefix></frame_prefix>
+    </plugin>
+  </gazebo>
 </robot>

Commit message: 更换pctplanner仓库，调整mid360朝向

File: src/unitree_go2w_ros2/go2w_description/urdf/go2w_description.urdf.xacro (robot description, xacro)
@@ -419,6 +419,5 @@
   <xacro:include filename="$(find go2w_description)/urdf/sensor/mid360_gpu.xacro"/>
   <xacro:mid360  name="livox_frame" parent="body" topic="/livox/lidar" imu_topic="/livox/imu" >
-    <!-- <origin xyz="0.3 0.0 0.10" rpy="0 0.5235987756 0"/> -->
-    <origin xyz="0.3 0.0 0.10" rpy="0 0.0 0"/>
+    <origin xyz="0.3 0.0 0.10" rpy="0 0 3.1415926"/>
   </xacro:mid360>
   <!-- Camera -->

File: src/unitree_go2w_ros2/go2w_description/urdf/go2w_description_gz.urdf.xacro (robot description, xacro)
@@ -313,5 +313,5 @@
     </inertial>
     <visual>
-      <origin xyz="0 0 0" rpy="0 0 ${PI}"/>
+      <origin xyz="0 0 0" rpy="0 0 0"/>
       <geometry>
         <mesh filename="${mesh_prefix}/mid-360-scaled.dae"/>
@@ -319,5 +319,5 @@
     </visual>
     <collision>
-      <origin xyz="0 0 0" rpy="0 0 ${PI}"/>
+      <origin xyz="0 0 0" rpy="0 0 0"/>
       <geometry>
         <mesh filename="${mesh_prefix}/mid-360-scaled.dae"/>
@@ -328,5 +328,5 @@
     <parent link="body"/>
     <child link="livox_frame"/>
-    <origin xyz="0.3 0.0 0.10" rpy="0 0 0"/>
+    <origin xyz="0.3 0.0 0.10" rpy="0 0 3.1415926"/>
   </joint>
   <xacro:macro name="joint_ros2_control_gz" params="prefix">

File: src/unitree_go2w_ros2/go2w_description/urdf/sensor/mid360_gpu.xacro (robot description, xacro)
@@ -24,5 +24,5 @@
     <link name="${name}">
       <visual>
-        <origin xyz="0 0 0" rpy="0 0 ${M_PI}"/>
+        <origin xyz="0 0 0" rpy="0 0 0"/>
         <geometry>
           <mesh filename="package://go2w_description/meshes/mid-360-scaled.dae"/>
@@ -30,5 +30,5 @@
       </visual>
       <collision>
-        <origin xyz="0 0 0" rpy="0 0 ${M_PI}"/>
+        <origin xyz="0 0 0" rpy="0 0 0"/>
         <geometry>
           <mesh filename="package://go2w_description/meshes/mid-360-scaled.dae"/>

Commit message: rl控制器可用

File: src/unitree_go2w_ros2/go2w_description/urdf/go2w_description.urdf.xacro (robot description, xacro)
@@ -419,5 +419,5 @@
   <xacro:include filename="$(find go2w_description)/urdf/sensor/mid360_gpu.xacro"/>
   <xacro:mid360  name="livox_frame" parent="body" topic="/livox/lidar" imu_topic="/livox/imu" >
-    <origin xyz="0.3 0.0 0.10" rpy="0 0 3.1415926"/>
+    <origin xyz="0.3 0.0 0.20" rpy="0 -0.5236 ${PI}"/>
   </xacro:mid360>
   <!-- Camera -->

File: src/unitree_go2w_ros2/go2w_description/urdf/go2w_description_gz.urdf.xacro (robot description, xacro)
@@ -328,5 +328,5 @@
     <parent link="body"/>
     <child link="livox_frame"/>
-    <origin xyz="0.3 0.0 0.10" rpy="0 0 3.1415926"/>
+    <origin xyz="0.3 0.0 0.10" rpy="0 -0.5236 ${PI}"/>
   </joint>
   <xacro:macro name="joint_ros2_control_gz" params="prefix">
@@ -365,4 +365,8 @@
     </joint>
     <joint name="${prefix}_foot_joint">
+      <command_interface name="effort">
+        <param name="min">${-foot_torque_max}</param>
+        <param name="max">${foot_torque_max}</param>
+      </command_interface>
       <command_interface name="velocity">
         <param name="min">${-foot_velocity_max}</param>
