Commit message: 增加imu自平衡

File: src/unitree_go2w_ros2/go2w_description/urdf/go2w_description_gz.urdf.xacro (robot description, xacro)
@@ -1,4 +1,5 @@
 <?xml version="1.0"?>
-<robot xmlns:xacro="http://ros.org/wiki/xacro" name="go2w_gz">
+<robot xmlns:xacro="http://ros.org/wiki/xacro" name="go2w">
+  <!-- Gloabal parameters -->
   <xacro:include filename="$(find go2w_description)/urdf/const.xacro"/>
   <xacro:property name="mesh_prefix" value="file://$(find go2w_description)/meshes" />
@@ -16,4 +17,5 @@
         <xacro:property name="left_sign" value="-1" />
     </xacro:if>
+    <!-- Hip -->
     <link name="${prefix}_hip">
       <inertial>
@@ -38,4 +40,5 @@
           <mesh filename="${mesh_prefix}/hip.dae" />
         </geometry>
+        <material name="深色橡胶_001-effect"><color rgba="0.6717055 0.6924257 0.7742702 1" /></material><material name="Material-effect"><color rgba="0.9 0.95 0.95 1" /></material>
       </visual>
       <collision>
@@ -59,4 +62,5 @@
       <dynamics damping="${hip_damping}" friction="${hip_friction}" />
     </joint>
+    <!-- Thigh -->
     <link name="${prefix}_thigh">
       <inertial>
@@ -75,4 +79,5 @@
           </xacro:if>
         </geometry>
+        <material name="深色橡胶_003-effect"><color rgba="0.6717055 0.6924257 0.7742702 1" /></material><material name="Material_009-effect"><color rgba="0.9 0.95 0.95 1" /></material>
       </visual>
       <collision>
@@ -91,4 +96,5 @@
       <dynamics damping="${thigh_damping}" friction="${thigh_friction}" />
     </joint>
+    <!-- Calf -->
     <link name="${prefix}_calf">
       <inertial>
@@ -107,4 +113,7 @@
             </xacro:if>
         </geometry>
+        <material name="">
+          <color rgba="1 1 1 1" />
+        </material>
       </visual>
       <collision>
@@ -123,4 +132,55 @@
       <dynamics damping="${calf_damping}" friction="${calf_friction}" />
     </joint>
+    <!-- Calf lower -->
+    <link name="${prefix}_calflower">
+      <collision>
+        <origin rpy="0 0 0" xyz="0 0 0" />
+        <geometry>
+            <cylinder length="${calf_lower_length}" radius="${calf_lower_radius}" />
+        </geometry>
+      </collision>
+    </link>
+    <joint name="${prefix}_calflower_joint" type="fixed">
+      <origin xyz="${calf_lower_offset_x} ${calf_lower_offset_y*left_sign} ${calf_lower_offset_z}" rpy="0 ${calf_lower_rotation_p} 0" />
+      <parent link="${prefix}_calf" />
+      <child link="${prefix}_calflower" />
+      <axis xyz="0 0 0" />
+    </joint>
+    <!-- Calf flower 1 -->
+    <link name="${prefix}_calflower1">
+      <collision>
+        <origin rpy="0 0 0" xyz="0 0 0" />
+        <geometry>
+            <cylinder length="${calf_lower1_length}" radius="${calf_lower1_radius}" />
+        </geometry>
+      </collision>
+    </link>
+    <joint name="${prefix}_calflower1_joint" type="fixed">
+      <origin xyz="${calf_lower1_offset_x} ${calf_lower1_offset_y*left_sign} ${calf_lower1_offset_z}" rpy="${calf_lower1_rotation_p}" />
+      <parent link="${prefix}_calflower" />
+      <child link="${prefix}_calflower1" />
+      <axis xyz="0 0 0" />
+    </joint>
+    <!-- Foot motor -->
+    <link name="${prefix}_foot_motor">
+      <inertial>
+        <origin xyz="${foot_motor_com_x} ${foot_motor_com_y} ${foot_motor_com_z}" rpy="0 0 0" />
+        <mass value="${foot_motor_mass}" />
+        <inertia ixx="${foot_motor_ixx}" ixy="${foot_motor_ixy*left_sign}" ixz="${foot_motor_ixz}" iyy="${foot_motor_iyy}" iyz="${foot_motor_iyz*left_sign}" izz="${foot_motor_izz}" />
+      </inertial>
+      <collision>
+        <origin rpy="${PI/2.0} 0 0" xyz="0 0 0" />
+        <geometry>
+            <cylinder length="${foot_motor_length}" radius="${foot_motor_radius}" />
+        </geometry>
+      </collision>
+    </link>
+    <joint name="${prefix}_foot_motor_joint" type="fixed">
+      <origin xyz="${foot_motor_offset_x} ${foot_motor_offset_y*left_sign} ${foot_motor_offset_z}" rpy="0 0.0 0" />
+      <parent link="${prefix}_calf" />
+      <child link="${prefix}_foot_motor" />
+      <axis xyz="0 0 0" />
+    </joint>
+    <!-- Foot -->
     <link name="${prefix}_foot">
       <inertial>
@@ -139,4 +199,7 @@
             </xacro:if>
         </geometry>
+        <material name="">
+          <color rgba="1 1 1 1" />
+        </material>
       </visual>
       <collision>
@@ -154,6 +217,12 @@
       <limit effort="${foot_torque_max}" velocity="${foot_velocity_max}" />
     </joint>
+    <gazebo reference="${prefix}_foot">
+        <mu1>3</mu1>
+        <mu2>3</mu2>
+    </gazebo>
   </xacro:macro>
+  <!-- Base-->
   <link name="base"/>
+  <!-- Body -->
   <link name="body">
     <inertial>
@@ -167,5 +236,5 @@
         <mesh filename="${mesh_prefix}/base.dae" />
       </geometry>
-    </visual>
+      <material name="深色橡胶_001-effect"><color rgba="0.6717055 0.6924257 0.7742702 1" /></material><material name="白色logo_001-effect"><color rgba="1 1 1 1" /></material><material name="黑色贴纸_007-effect"><color rgba="0.009018 0.009018 0.009018 1" /></material><material name="黑色金属_007-effect"><color rgba="0.01341 0.01341 0.01341 1" /></material><material name="黑色塑料_003-effect"><color rgba="0.023455 0.023455 0.023455 1" /></material></visual>
     <collision>
       <origin rpy="0 0 0" xyz="0 0 0" />
@@ -179,4 +248,5 @@
     <child link="body" />
   </joint>
+  <!-- Head Upper-->
   <link name="Head_upper">
     <inertial>
@@ -198,4 +268,5 @@
     <axis xyz="0 0 0" />
   </joint>
+  <!-- Head Lower -->
   <link name="Head_lower">
     <inertial>
@@ -221,4 +292,5 @@
   <xacro:leg prefix="RL" front="False" left="True"/>
   <xacro:leg prefix="RR" front="False" left="False"/>
+  <!-- IMU -->
   <link name="imu">
     <inertial>

Commit message: sync

File: src/unitree_go2w_ros2/go2w_description/urdf/go2w_description_gz.urdf.xacro (robot description, xacro)
@@ -328,5 +328,5 @@
     <parent link="body"/>
     <child link="livox_frame"/>
-    <origin xyz="0.3 0.0 0.10" rpy="0 -0.5236 ${PI}"/>
+    <origin xyz="0.3 0.0 0.20" rpy="0 -0.5236 ${PI}"/>
   </joint>
   <xacro:macro name="joint_ros2_control_gz" params="prefix">
